File: pierce.kicad_pcb (KiCad board)
At the start: 2 copper layers, 275.7 x 105.8 mm, 81 parts, among them J1 Conn_01x10, J2 Conn_01x10, J3 Trackpoint, SW1 SW_PUSH, SW10 SW_PUSH, SW11 SW_PUSH, SW12 SW_PUSH, SW13 SW_PUSH, SW14 SW_PUSH, SW15 SW_PUSH, SW16 SW_PUSH, SW17 SW_PUSH, SW18 SW_PUSH, SW19 SW_PUSH, SW2 SW_PUSH, SW20 SW_PUSH, SW21 SW_PUSH, SW22 SW_PUSH, SW23 SW_PUSH, SW24 SW_PUSH, SW25 SW_PUSH, SW26 SW_PUSH, SW27 SW_PUSH, SW28 SW_PUSH, SW29 SW_PUSH, SW3 SW_PUSH, SW30 SW_PUSH, SW31 SW_PUSH, SW32 SW_PUSH, SW33 SW_PUSH, SW34 SW_PUSH, SW35 SW_PUSH, SW36 SW_PUSH, SW37 SW_PUSH, SW4 SW_PUSH, SW5 SW_PUSH, SW6 SW_PUSH, SW7 SW_PUSH, SW8 SW_PUSH, SW9 SW_PUSH, U1 ProMicro_r

Commit message: v 0.2
Parts:
- added Ref**: Val**, kbd:M2_Threads_v2, F.Cu at (153.8, 67.6)
- D1, D10, D11, D12, D13, D14, D15, D16, D17, D18, D19, D2, D20, D21, D22, D23, D24, D25, D26, D27, D28, D29, D3, D30, D31, D32, D33, D34, D35, D36, D4, D5, D6, D7, D8, D9: moved to B.Cu
- J1, J2: value Conn_01x10 -> Conn_02x05
- moved R2 140.6 mm to (161.6, 53.2)
- moved D4 130.1 mm to (189.5, 30.6), turned to 270 degrees
- moved R1 129.1 mm to (161.8, 56.5)
- moved R3 128.4 mm to (161.6, 47.1)
- moved D7 119.6 mm to (179.2, 98.2), turned to 270 degrees
- moved D5 115.3 mm to (189.5, 48.1), turned to 270 degrees
- moved C1 114.2 mm to (161.6, 50.4)
- moved D11 113.8 mm to (208.7, 28.0), turned to 270 degrees
- moved D18 102.9 mm to (139.9, 85.0), turned to 180 degrees
- moved D6 101.3 mm to (189.4, 66.9), turned to 270 degrees
- moved D34 101.0 mm to (257.1, 39.4)
- moved D26 98.5 mm to (135.8, 90.5), turned to 240 degrees
- moved D30 97.5 mm to (108.9, 29.6), turned to 270 degrees
- moved D14 97.4 mm to (198.6, 95.4), turned to 90 degrees
- moved D13 97.1 mm to (208.7, 64.4), turned to 270 degrees
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Other:
- board size 275.7 x 105.8 mm -> 236.3 x 105.8 mm
- board text added: "NOTE DIRECTION"

Commit message: Routed right half
Parts:
- added Ref**: Val**, kbd:M2_Threads_v2, F.Cu at (153.9, 30.3)
- added Ref**: Val**, kbd:M2_Threads_v2, F.Cu at (167.1, 30.3)
- added Ref**: Val**, kbd:M2_Threads_v2, F.Cu at (165.2, 72.9)
- C1, R1, R2, R3: moved to B.Cu
- moved D19 14.6 mm to (213.2, 25.5)
- moved D11 14.5 mm to (194.3, 27.1)
- moved D20 14.3 mm to (213.3, 42.5)
- moved D21 14.3 mm to (213.4, 61.1)
- moved D13 14.2 mm to (194.5, 64.5)
- moved D12 14.2 mm to (194.4, 45.6)
- moved D5 14.1 mm to (175.4, 47.8)
- moved D29 14.1 mm to (232.5, 64.4)
- moved D6 14.1 mm to (175.3, 67.0)
- moved D4 13.9 mm to (175.6, 30.9)
- moved D28 13.8 mm to (232.4, 44.9)
- moved D27 12.1 mm to (232.4, 26.9)
- moved R3 11.9 mm to (161.6, 35.2)
- moved C1 11.7 mm to (161.6, 38.7)
- moved SW37 11.6 mm to (229.1, 86.7)
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Routing:
- net row1: track 0.00 -> 229.3 mm, vias 0 -> 2
- net row0: track 0.00 -> 228.7 mm, vias 0 -> 2
- net reset: track 0.00 -> 211.8 mm
- net row2: track 0.00 -> 164.5 mm, vias 0 -> 2
- net col9: track 0.00 -> 139.9 mm, vias 0 -> 2
- net col7: track 0.00 -> 134.1 mm, vias 0 -> 5
- net col8: track 0.00 -> 123.4 mm, vias 0 -> 3
- net col6: track 0.00 -> 118.2 mm, vias 0 -> 5
- net col5: track 0.00 -> 110.5 mm, vias 0 -> 4
- net row3: track 0.00 -> 108.6 mm
- net SDA: track 0.00 -> 57.3 mm
- net VCC: track 0.00 -> 54.3 mm, vias 0 -> 1
- net Net-(C1-Pad2): track 0.00 -> 41.7 mm, vias 0 -> 1
- net SCL: track 0.00 -> 40.1 mm
- net col4: track 0.00 -> 34.9 mm, vias 0 -> 1
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Other:
- board size 236.3 x 105.8 mm -> 275.5 x 105.6 mm
- board text added: "100k"
- board text added: "2.2uF"
- board text added: "4k7"

Commit message: Finished routing (improved routing from last commit)
Parts:
- removed the Ref** at (153.9, 30.3)
- removed the Ref** at (167.1, 30.3)
- removed the Ref** at (165.2, 72.9)
- removed the Ref** at (153.8, 67.6)
- added Ref**: Val**, kbd:M2_HOLE_v2, F.Cu at (117.7, 91.9)
- added Ref**: Val**, kbd:M2_Threads_v2, F.Cu at (167.0, 72.6)
- added Ref**: Val**, kbd:M2_HOLE_v2, F.Cu at (71.6, 81.2)
- added Ref**: Val**, kbd:M2_HOLE_v2, F.Cu at (47.8, 54.2)
- added Ref**: Val**, kbd:M2_HOLE_v2, F.Cu at (104.7, 43.0)
- added Ref**: Val**, kbd:M2_HOLE_v2, F.Cu at (175.9, 85.2)
- added Ref**: Val**, kbd:M2_HOLE_v2, F.Cu at (224.4, 82.5)
- added Ref**: Val**, kbd:M2_HOLE_v2, F.Cu at (247.6, 54.2)
- added Ref**: Val**, kbd:M2_HOLE_v2, F.Cu at (190.7, 43.0)
- added Ref**: Val**, kbd:M2_Threads_v2, F.Cu at (153.9, 68.0)
- J1, J2: value Conn_02x05 -> Conn_01x10
- SW1, SW10, SW11, SW12, SW13, SW14, SW15, SW16, SW17, SW18, SW19, SW2, SW20, SW21, SW22, SW23, SW24, SW25, SW26, SW27, SW28, SW29, SW3, SW30, SW31, SW32, SW33, SW34, SW35, SW36, SW4, SW5, SW6, SW7, SW8, SW9: footprint kbd:CherryMX_Hotswap -> kbd:CherryMX_ChocV2_1u
- moved D18 43.3 mm to (96.6, 84.6)
- moved D14 31.2 mm to (168.3, 88.0), turned to 270 degrees
- moved D33 19.8 mm to (120.5, 84.8), turned to 270 degrees
- moved D26 19.2 mm to (117.5, 84.8), turned to 270 degrees
- moved D7 17.2 mm to (165.3, 88.0)
- moved D25 17.1 mm to (103.6, 70.3)
- moved D24 16.9 mm to (103.6, 51.3), turned to 90 degrees
- moved D9 16.8 mm to (65.6, 51.3), turned to 90 degrees
- moved D23 16.7 mm to (103.6, 32.3), turned to 90 degrees
- moved D20 16.5 mm to (227.2, 51.3), turned to 90 degrees
- moved D10 16.2 mm to (65.6, 70.3)
- moved D19 15.5 mm to (227.2, 32.3), turned to 90 degrees
- moved D21 15.4 mm to (227.2, 68.0)
- moved D8 14.4 mm to (65.6, 32.3), turned to 90 degrees
- moved D6 14.2 mm to (189.2, 69.8)
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Connections:
- J1 pad 1: row0l -> row2l
- J1 pad 10: col4l -> col0l
- J1 pad 2: row1l -> row0l
- J1 pad 3: row2l -> row1l
- J1 pad 4: row3l -> col3l
- J1 pad 5: (no net) -> row3l
- J1 pad 6: col0l -> col2l
- J1 pad 7: col1l -> (no net)
- J1 pad 8: col2l -> col1l
- J1 pad 9: col3l -> col4l
- J2 pad 1: row0 -> row2
- J2 pad 10: col4 -> col0
- J2 pad 2: row1 -> row0
- J2 pad 3: row2 -> row1
- J2 pad 4: row3 -> col3
- J2 pad 5: (no net) -> row3
- J2 pad 6: col0 -> col2
- J2 pad 7: col1 -> (no net)
- J2 pad 8: col2 -> col1
- J2 pad 9: col3 -> col4
- U1 pad 10: col7 -> col6
- U1 pad 11: col8 -> col5
- U1 pad 12: col9 -> col4
- U1 pad 7: col4 -> col9
- U1 pad 8: col5 -> col8
- U1 pad 9: col6 -> col7
Routing:
- net col0l: track 0.00 -> 160.3 mm, vias 0 -> 1
- net col2l: track 0.00 -> 136.8 mm, vias 0 -> 1
- net col1l: track 0.00 -> 134.3 mm, vias 0 -> 1
- net row0l: track 0.00 -> 122.5 mm, vias 0 -> 1
- net row2l: track 0.00 -> 117.2 mm
- net col3l: track 0.00 -> 114.4 mm, vias 0 -> 2
- net row1l: track 0.00 -> 101.8 mm, vias 0 -> 1
- net col4l: track 0.00 -> 80.7 mm
- net row1: track 229.3 -> 159.7 mm, vias 2 -> 3
- net row0: track 228.7 -> 179.7 mm, vias 2 -> 0
- net Net-(D33-Pad2): track 0.00 -> 29.9 mm
- net row3l: track 0.00 -> 29.8 mm
- net Net-(D14-Pad2): track 9.45 -> 35.0 mm
- net Net-(D3-Pad2): track 0.00 -> 25.4 mm
- net Net-(D2-Pad2): track 0.00 -> 25.4 mm
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- added copper zone on B.Cu, net GND
- added copper zone on F.Cu, net GND
Other:
- outline, holes or cut-outs redrawn
- board text added: "Pierce 1.0 Design by Durken"
- board text removed: "NOTE DIRECTION"

Commit message: Adjusted text on silk layer
Parts:
- added REF**: Breakaway_Tabs, kbd:Breakaway_Tabs, F.Cu at (101.3, 26.0)
- added REF**: Breakaway_Tabs, kbd:Breakaway_Tabs, F.Cu at (63.3, 26.0)
- added REF**: Breakaway_Tabs, kbd:Breakaway_Tabs, F.Cu at (62.9, 95.0)
- added REF**: Breakaway_Tabs, kbd:Breakaway_Tabs, F.Cu at (195.9, 26.0)
- added REF**: Breakaway_Tabs, kbd:Breakaway_Tabs, F.Cu at (233.9, 26.0)
- added REF**: Breakaway_Tabs, kbd:Breakaway_Tabs, F.Cu at (234.2, 95.0)
- moved SW10 6.30 mm to (63.2, 73.2)
- moved D26 6.30 mm to (123.1, 87.8)
- moved D33 6.30 mm to (126.1, 87.8)
- moved Ref** 6.30 mm to (123.3, 94.9)
- moved Ref** 6.30 mm to (77.2, 84.2)
- moved SW18 6.30 mm to (92.2, 93.1)
- moved SW33 6.30 mm to (132.8, 103.7)
- moved D1 6.30 mm to (52.2, 47.7)
- moved D2 6.30 mm to (52.2, 66.7)
- moved SW1 6.30 mm to (44.2, 47.7)
- moved SW2 6.30 mm to (44.2, 66.7)
- moved D10 6.30 mm to (71.2, 73.2)
- moved D17 6.30 mm to (74.2, 73.2)
- moved D18 6.30 mm to (102.2, 87.5)
- moved D25 6.30 mm to (109.2, 73.2)
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Other:
- board size 275.5 x 105.6 mm -> 227.3 x 105.6 mm
- board text added: "Pierce 1.0"
- board text removed: "Pierce 1.0 Design by Durken"
