File: pcb/_autosave-pierce.kicad_pcb (KiCad board)
At the start: 2 copper layers, 227.3 x 105.6 mm, 81 parts, among them J1 Conn_01x10, J2 Conn_01x10, J3 Trackpoint, SW1 SW_PUSH, SW10 SW_PUSH, SW11 SW_PUSH, SW12 SW_PUSH, SW13 SW_PUSH, SW14 SW_PUSH, SW15 SW_PUSH, SW16 SW_PUSH, SW17 SW_PUSH, SW18 SW_PUSH, SW19 SW_PUSH, SW2 SW_PUSH, SW20 SW_PUSH, SW21 SW_PUSH, SW22 SW_PUSH, SW23 SW_PUSH, SW24 SW_PUSH, SW25 SW_PUSH, SW26 SW_PUSH, SW27 SW_PUSH, SW28 SW_PUSH, SW29 SW_PUSH, SW3 SW_PUSH, SW30 SW_PUSH, SW31 SW_PUSH, SW32 SW_PUSH, SW33 SW_PUSH, SW34 SW_PUSH, SW35 SW_PUSH, SW36 SW_PUSH, SW37 SW_PUSH, SW4 SW_PUSH, SW5 SW_PUSH, SW6 SW_PUSH, SW7 SW_PUSH, SW8 SW_PUSH, SW9 SW_PUSH, U1 Elite-C_reverse

Commit message: Changed footprint to Elite-C (Reversed for flipped mounting) Changed pins connected to trackpoint to allow USART. (CLK-D5, SDA-D2) Rearranged connection order of trackpoint to match R61 module Cleaner routing
Changed lines of the file:
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@@
     (thickness 1.6)
     (drawings 713)
-    (tracks 768)
+    (tracks 767)
     (zones 0)
     (modules 81)
@@
   (segment (start 128.38 97.274852) (end 128.38 88.2) (width 0.25) (layer F.Cu) (net 51))
   (segment (start 165.2584 66.88) (end 165.2664 66.872) (width 0.25) (layer B.Cu) (net 52))
-  (segment (start 165.258 51.632) (end 165.2664 51.632) (width 0.25) (layer B.Cu) (net 0))
   (segment (start 153.82501 70.77499) (end 152.6 72) (width 0.5) (layer F.Cu) (net 1))
   (segment (start 153.82501 50.54101) (end 153.82501 70.77499) (width 0.5) (layer F.Cu) (net 1))
