File: pcb/wireless/pierce.sch (KiCad schematic (older format))
At the start: 23 parts, among them SW1 SW_PUSH, SW10 SW_PUSH, SW15 SW_PUSH, SW16 SW_PUSH, SW17 SW_PUSH, SW18 SW_PUSH, SW2 SW_PUSH, SW23 SW_PUSH, SW24 SW_PUSH, SW25 SW_PUSH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

Commit message: small adjustments
Connections:
- no-connect marks 0 -> 25
Changed lines of the file:
@@
 encoding utf-8
 Sheet 1 1
-Title "pierce keyboard - wireless"
+Title "pierce keyboard - wireless side"
 Date "2021-06-16"
 Rev "v 2.0"
@@
 	1    0    0    -1
 $EndComp
-Wire Wire Line
-	8400 1400 8400 1500
 $Comp
 L power:GND #PWR027
@@
 L power:GND #PWR025
 U 1 1 60D91507
-P 8400 1500
-F 0 "#PWR025" H 8400 1250 50  0001 C CNN
-F 1 "GND" H 8405 1327 50  0000 C CNN
-F 2 "" H 8400 1500 50  0001 C CNN
-F 3 "" H 8400 1500 50  0001 C CNN
-	1    8400 1500
+P 8400 1400
+F 0 "#PWR025" H 8400 1150 50  0001 C CNN
+F 1 "GND" V 8400 1200 50  0000 C CNN
+F 2 "" H 8400 1400 50  0001 C CNN
+F 3 "" H 8400 1400 50  0001 C CNN
+	1    8400 1400
 	1    0    0    -1
 $EndComp
@@
 	1    0    0    -1
 $EndComp
-Wire Wire Line
-	8700 1500 8700 1400
 $Comp
 L power:VCC #PWR026
 U 1 1 60DA0767
-P 8700 1500
-F 0 "#PWR026" H 8700 1350 50  0001 C CNN
-F 1 "VCC" H 8715 1673 50  0000 C CNN
-F 2 "" H 8700 1500 50  0001 C CNN
-F 3 "" H 8700 1500 50  0001 C CNN
-	1    8700 1500
+P 8700 1400
+F 0 "#PWR026" H 8700 1250 50  0001 C CNN
+F 1 "VCC" V 8700 1600 50  0000 C CNN
+F 2 "" H 8700 1400 50  0001 C CNN
+F 3 "" H 8700 1400 50  0001 C CNN
+	1    8700 1400
 	-1   0    0    1
 $EndComp
@@
 Text GLabel 7700 2300 2    50   Input ~ 0
 SW34L
+NoConn ~ 5800 1800
+NoConn ~ 5800 1900
+NoConn ~ 5800 2000
+NoConn ~ 5800 2100
+NoConn ~ 7700 1400
+NoConn ~ 7700 1500
+NoConn ~ 7700 1600
+NoConn ~ 7700 1700
+NoConn ~ 7700 2000
+NoConn ~ 7700 2100
+NoConn ~ 7700 2200
+NoConn ~ 7700 2400
+NoConn ~ 7700 2500
+NoConn ~ 7750 4500
+NoConn ~ 7750 4600
+NoConn ~ 7750 4900
+NoConn ~ 7750 5000
+NoConn ~ 5850 4700
+NoConn ~ 5850 4600
+NoConn ~ 5850 4500
+NoConn ~ 5850 4400
+NoConn ~ 5850 4300
+NoConn ~ 5850 4200
+NoConn ~ 5850 4100
+NoConn ~ 5850 4000
 $EndSCHEMATC
