File: pcb/wireless/pierce.kicad_pcb (KiCad board)
At the start: 2 copper layers, 112.2 x 91.4 mm, 29 parts, among them SW1 SW_PUSH, SW10 SW_PUSH, SW15 SW_PUSH, SW16 SW_PUSH, SW17 SW_PUSH, SW18 SW_PUSH, SW2 SW_PUSH, SW23 SW_PUSH, SW24 SW_PUSH, SW25 SW_PUSH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

Commit message: small adjustments
Parts:
- removed REF** (x2): OSHW-Logo2_7.3x6mm_SilkScreen, pierce:OSHW-Logo2_7.3x6mm_SilkScreen
Other:
- outline, holes or cut-outs redrawn
