File: pcb/wired/pierce.kicad_pcb (KiCad board)
At the start: 2 copper layers, 115 x 91.4 mm, 39 parts, among them SW11 SW_PUSH, SW12 SW_PUSH, SW13 SW_PUSH, SW14 SW_PUSH, SW19 SW_PUSH, SW20 SW_PUSH, SW21 SW_PUSH, SW22 SW_PUSH, SW27 SW_PUSH, SW28 SW_PUSH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

Commit message: schematic done, started place & route
Parts:
- removed AVR1: Elite-C_reverse, pierce:Elite-C_reverse_D5
- added C2: 22p, Capacitor_SMD:C_0805_2012Metric_Pad1.18x1.45mm_HandSolder, F.Cu at (127.6, 39.8)
- added C3: 100n, Capacitor_SMD:C_0805_2012Metric_Pad1.18x1.45mm_HandSolder, B.Cu at (169.1, 49.8)
- added C4: 100n, Capacitor_SMD:C_0805_2012Metric_Pad1.18x1.45mm_HandSolder, F.Cu at (151.1, 61.8)
- added C5: 22p, Capacitor_SMD:C_0805_2012Metric_Pad1.18x1.45mm_HandSolder, B.Cu at (165.1, 44.8)
- added C6: 100n, Capacitor_SMD:C_0805_2012Metric_Pad1.18x1.45mm_HandSolder, B.Cu at (150.1, 56.3)
- added C7: 100n, Capacitor_SMD:C_0805_2012Metric_Pad1.18x1.45mm_HandSolder, B.Cu at (150.1, 51.3)
- added C8: 10u, Capacitor_SMD:C_0805_2012Metric_Pad1.18x1.45mm_HandSolder, B.Cu at (169.1, 54.3)
- added C9: 1u, Capacitor_SMD:C_0805_2012Metric_Pad1.18x1.45mm_HandSolder, F.Cu at (140.6, 37.8)
- added F1: 500m, Fuse:Fuse_0805_2012Metric_Pad1.15x1.40mm_HandSolder, F.Cu at (159.6, 44.3)
- added J1: AVR-ISP-6, random-keyboard-parts:Reset_Pretty-Mask, F.Cu at (125.8, 49.4)
- added R10: 10k, Resistor_SMD:R_0805_2012Metric_Pad1.20x1.40mm_HandSolder, F.Cu at (115.1, 38.3)
- added R11: 10k, Resistor_SMD:R_0805_2012Metric_Pad1.20x1.40mm_HandSolder, F.Cu at (111.6, 33.3)
- added R6: 5.1k, Resistor_SMD:R_0805_2012Metric_Pad1.20x1.40mm_HandSolder, F.Cu at (151.1, 40.3)
- added R7: 5.1k, Resistor_SMD:R_0805_2012Metric_Pad1.20x1.40mm_HandSolder, F.Cu at (162.1, 40.3)
- added R8: 22, Resistor_SMD:R_0805_2012Metric_Pad1.20x1.40mm_HandSolder, F.Cu at (131.3, 52.9)
- added R9: 22, Resistor_SMD:R_0805_2012Metric_Pad1.20x1.40mm_HandSolder, F.Cu at (134.1, 38.3)
- added U1: PRTR5V0U2X, random-keyboard-parts:SOT143B, F.Cu at (154.6, 44.3)
- added U2: ATmega32U4-AU, Package_QFP:TQFP-44_10x10mm_P0.8mm, B.Cu at (159.1, 53.8)
- added USB1: HRO-TYPE-C-31-M-12, Type-C:HRO-TYPE-C-31-M-12-HandSoldering, F.Cu at (157.1, 27.8)
- added Y1: XTAL, Crystal:Crystal_SMD_3225-4Pin_3.2x2.5mm_HandSoldering, F.Cu at (111.6, 52.1)
- YJR1: value YJ14015 -> YJ-14015-NRF51822
- moved R1 31.2 mm to (173.5, 64.9), turned to 90 degrees
- moved R2 30.9 mm to (183.3, 64.9), turned to 90 degrees
- moved C1 30.4 mm to (176.7, 64.9), turned to 90 degrees
- moved R3 30.3 mm to (180.0, 64.9), turned to 90 degrees
- moved R5 26.4 mm to (154.4, 79.9), turned to 270 degrees
- moved R4 23.0 mm to (157.7, 79.9), turned to 270 degrees
Routing:
- net reset: track 127.5 -> 67.6 mm
- net I2C_SDA: track 38.9 -> 0.03 mm, vias 1 -> 0
- net VCC_5V: track 67.9 -> 29.4 mm
- net SDA: track 36.0 -> 0.00 mm, vias 2 -> 0
- net I2C_SCL: track 35.2 -> 0.00 mm, vias 1 -> 0
- net Net-(C1-Pad2): track 31.3 -> 0.00 mm
- net SCL: track 22.2 -> 0.00 mm
- net VCC_3.3V: track 121.7 -> 101.2 mm
